File: saw-animator.kicad_pcb (KiCad board)
At the start: 2 copper layers, 50.5 x 89.7 mm, 63 parts, among them J1 Conn_02x05_Odd_Even, J10 AudioJack2_SwitchT, J2 Conn_01x03_Socket, J3 Conn_01x03_Socket, J4 Conn_01x03_Socket, J5 Conn_01x03_Pin, J6 Conn_01x03_Pin, J7 Conn_01x03_Pin, J8 AudioJack2_SwitchT, J9 AudioJack2_SwitchT, Q1 BC547, U1 TL074, U2 TL074

Commit message: fix: updating resistances to easily obtainable values
Parts:
- D6: value LED -> LED_GREEN
- R15: value 47K -> 120K
- R16: value 88K -> 220K
Changed lines of the file:
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@@
         (effects (font (size 1 1) (thickness 0.15)))
     )
-    (fp_text value "LED" (at 1.27 2.96) (layer "F.Fab")
+    (fp_text value "LED_GREEN" (at 1.27 2.96) (layer "F.Fab")
         (effects (font (size 1 1) (thickness 0.15)))
     )
@@
         (effects (font (size 1 1) (thickness 0.15)) (justify mirror))
     )
-    (fp_text value "47K" (at 0 -1.65) (layer "B.Fab")
+    (fp_text value "120K" (at 0 -1.65) (layer "B.Fab")
         (effects (font (size 1 1) (thickness 0.15)) (justify mirror))
     )
@@
         (effects (font (size 1 1) (thickness 0.15)) (justify mirror))
     )
-    (fp_text value "88K" (at 0 -1.65) (layer "B.Fab")
+    (fp_text value "220K" (at 0 -1.65) (layer "B.Fab")
         (effects (font (size 1 1) (thickness 0.15)) (justify mirror))
     )
@@
     (descr "SOIC, 14 Pin (JEDEC MS-012AB, https://www.analog.com/media/en/package-pcb-resources/package/pkg_pdf/soic_narrow-r/r_14.pdf), generated with kicad-footprint-generator ipc_gullwing_generator.py")
     (tags "SOIC SO")
-    (property "Sheetfile" "saw-animator.kicad_sch")
-    (property "Sheetname" "")
+    (property "PartNum" "595-TL074CDR")
+    (property "Sheetfile" "saw-animator.kicad_sch")
+    (property "Sheetname" "")
+    (property "Vendor" "Mouser")
     (property "ki_description" "Quad Low-Noise JFET-Input Operational Amplifiers, DIP-14/SOIC-14")
     (property "ki_keywords" "quad opamp")
@@
     (descr "SOIC, 14 Pin (JEDEC MS-012AB, https://www.analog.com/media/en/package-pcb-resources/package/pkg_pdf/soic_narrow-r/r_14.pdf), generated with kicad-footprint-generator ipc_gullwing_generator.py")
     (tags "SOIC SO")
-    (property "Sheetfile" "saw-animator.kicad_sch")
-    (property "Sheetname" "")
+    (property "PartNum" "595-TL074CDR")
+    (property "Sheetfile" "saw-animator.kicad_sch")
+    (property "Sheetname" "")
+    (property "Vendor" "Mouser")
     (property "ki_description" "Quad Low-Noise JFET-Input Operational Amplifiers, DIP-14/SOIC-14")
     (property "ki_keywords" "quad opamp")
